File: fase3_pcb/v7/v7_drone.kicad_pcb (KiCad board)
At the start: 4 copper layers, 220 x 160 mm, 319 parts, among them J1 AMASS, J2 USB, Q1 TO-252-2, SW1 SW, SW2 SW, U10 SOIC-16, U11 SOIC-16, U8 SOIC-16, U9 SOIC-16

Commit message: fix(v10): auditoria independente — 9 bloqueadores corrigidos com prova E2E
AUDITORIA (AUDITORIA_ERROS_2026-10-04.md): ~110 erros, 9 críticos, 3 alegações
do ERROS_CONHECIDOS refutadas (1.g parcial, 3.3, 7).

Fase 3 v10 (gera_pcb_v10.py + verifica_fase3_v10.py):
- packer: sinal dx/dy corrigido (eram 27 footprints/199 pads FORA do contorno,
  14 curtos pad×pad) e bbox por PADS (a antiga media texto de silkscreen)
- keepout da borda superior adicionado; acha_via respeita keepout+clearance
- zonas para VBAT/VBAT_F/PHM*/SNM (o 1.g era falso p/ 26 nets: 30 A sem cobre)
- gates novos G1-G7: v10 = G1-G5/G7 OK (G6=18 pads documentado)

Netlist (gera_pcb_v7.py): typo RBM###/RB_M### desconectava as 12 entradas BEMF
do ADC; ferrite 3V3_A_F orfão virou 3V3_IMU (IMU+baro). 0 nets de 1 pad.

Pipeline FreeRouting — bug 1.h RESOLVIDO (dsn_export.py):
- P1 0==False: todo pad virava círculo Ø=max(w,h) -> blobs selados
- P2 (via VIA1) nunca declarada -> board sem nenhuma via
- P3 rotação dupla; P4 pins duplicados (~39k); P5 THT mult-camada
- PROVA corte 16 módulos: 46 wires/8 vias/9 nets (antes 0 em 0,82 s fake)
- PROVA placa completa: 49min47s reais, SES 252 KB, 1410 wires, 404 vias,
  149/151 nets, 3909 trilhas importadas (v10_roteada.kicad_pcb)
- ses_import.py: 4 bugs latentes corrigidos (GetNetCode, PCB_TRACK/PCB_VIA,
  walk_net aninhado) — nunca tinha completado 1 execução

Firmware: API ESP-IDF v5.4 real (F1), 20 kHz exatos (F2), canal LEDC (F3),
protocolo MCP3208 (F4), init chamados (F5), GPIOs reais no board_pins.h
(RF-07 refutada), FREERTOS_HZ=1000 — ver firmware/RESUMO_CORRECOES_2026-10-04.md

Fase 0: 25 correções de cálculo executadas (Psw 2x, perdas 16x, BEMF 2,74 V,
IPC interno 42,6 mm, Ciss 12 nF, E_oss com 1/2, L7 estourado honestamente,
margem do MOSFET 85,2 V > 80 V = FALHA documentada) + 6 saídas regeneradas.

BOM_FABRICACAO_v10.csv: MOSFET NVMFS6H824NT1G (o antigo comprava IPB017N10N5
TO-263-7, incompatível), ADC 4x MCP3208 (o que o board tem), separadores.

Pendênci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
Connections:
- CIMU pad 1: 3V3 -> 3V3_IMU
- CbeM101 pad 1: RBM101 -> RB_M101
- CbeM102 pad 1: RBM102 -> RB_M102
- CbeM103 pad 1: RBM103 -> RB_M103
- CbeM201 pad 1: RBM201 -> RB_M201
- CbeM202 pad 1: RBM202 -> RB_M202
- CbeM203 pad 1: RBM203 -> RB_M203
- CbeM301 pad 1: RBM301 -> RB_M301
- CbeM302 pad 1: RBM302 -> RB_M302
- CbeM303 pad 1: RBM303 -> RB_M303
- CbeM401 pad 1: RBM401 -> RB_M401
- CbeM402 pad 1: RBM402 -> RB_M402
- CbeM403 pad 1: RBM403 -> RB_M403
- FLDO pad 2: 3V3_A_F -> 3V3_IMU
- Rb1M101 pad 2: RBM101 -> RB_M101
- Rb1M102 pad 2: RBM102 -> RB_M102
- Rb1M103 pad 2: RBM103 -> RB_M103
- Rb1M201 pad 2: RBM201 -> RB_M201
- Rb1M202 pad 2: RBM202 -> RB_M202
- Rb1M203 pad 2: RBM203 -> RB_M203
- Rb1M301 pad 2: RBM301 -> RB_M301
- Rb1M302 pad 2: RBM302 -> RB_M302
- Rb1M303 pad 2: RBM303 -> RB_M303
- Rb1M401 pad 2: RBM401 -> RB_M401
- Rb1M402 pad 2: RBM402 -> RB_M402
- Rb1M403 pad 2: RBM403 -> RB_M403
- Rb2M101 pad 1: RBM101 -> RB_M101
- Rb2M102 pad 1: RBM102 -> RB_M102
- Rb2M103 pad 1: RBM103 -> RB_M103
- Rb2M201 pad 1: RBM201 -> RB_M201
- Rb2M202 pad 1: RBM202 -> RB_M202
- Rb2M203 pad 1: RBM203 -> RB_M203
- Rb2M301 pad 1: RBM301 -> RB_M301
- Rb2M302 pad 1: RBM302 -> RB_M302
- Rb2M303 pad 1: RBM303 -> RB_M303
- Rb2M401 pad 1: RBM401 -> RB_M401
- Rb2M402 pad 1: RBM402 -> RB_M402
- Rb2M403 pad 1: RBM403 -> RB_M403
- U_BARO pad CSB: 3V3 -> 3V3_IMU
- U_BARO pad VDD: 3V3 -> 3V3_IMU
- U_BARO pad VDDIO: 3V3 -> 3V3_IMU
- U_IMU pad 5: 3V3 -> 3V3_IMU
- U_IMU pad 8: 3V3 -> 3V3_IMU
