File: fase3_pcb/v10/v10_drone.kicad_pcb (KiCad board)
At the start: 6 copper layers, 190 x 145 mm, 319 parts, among them J1 AMASS, J2 USB, Q1 TO-252-2, SW1 SW, SW2 SW, U10 SOIC-16, U11 SOIC-16, U8 SOIC-16, U9 SOIC-16

Commit message: fix(v10): auditoria 12/10 - 354 curtos cobre-excluido + G6 completo + gate G8 + harness
Auditoria independente no 2 (mesmas ferramentas: pcbnew 5.1.9, fonte do FR,
pipeline executado de verdade). Evidencia completa: ERROS_CONHECIDOS.md secao 9.

- CRITICO: a roteagem v10 tinha 354 violacoes trilha x cobre de net excluida
  (medição exata segmento x retangulo rotacionado; d ate -0,93 mm): o DSN
  omite as 28 nets de potencia e o roteador NAO via os pads/vias de stitch
  delas. dsn_export.py agora exporta cada pad/via excluido como
  (keepout (rectangle LAYER ...)) - 3.167 scopes, import zero warnings.
  Re-roteamento completo em andamento com o DSN novo.
- CRITICO: o board commitado em f58c376 estava STALE vs o proprio gerador
  (o fix G6 do codigo nunca foi re-executado; a verificacao 18-pads era da
  rodada anterior). Regenerado: +51 vias de stitch.
- G6 fechado no gerador: 3a passada com colisao retangular borda-a-borda
  + isencao de mesma-net (via-in-pad GND e' pratica padrao de stitch) +
  conferencia de via compartilhada <=1,6 mm (U_IMU.7 ja' estava a 0,90 mm
  da via do U_IMU.9; U_LDO.GND resgatada com busca precisa).
  Base regenerada: TODOS OS GATES OK (G1-G8).
- Gate novo G8 no verificador: trilha x cobre-excluido = 0 violacoes,
  distancia exata (projecao alternada segmento x retangulo rotacionado).
  No board roteado antigo: 354 [FALHA] - o gate que teria pego tudo.
- verificacoes/verifica_projeto.py: o "Proximo passo" do ERROS_CONHECIDOS
  finalmente construido - assercoes duras (SES wires/vias/cobertura,
  gates G1-G8 na base E no roteado, cobertura de rota, BOM compravel).
  Exit 1 com a lista exata do que falta: 'pronto' e' do artefato.
- fr_watchdog.py: 2x S110 try-except-pass agora logam (lint do `concise`).
- FONTE_FREEROUTING.md: secao keepouts + bug 0-wires marcado SUPERSEDED.
Routing:
- net VBAT_PROT: vias 51 -> 68
- net GND: vias 347 -> 381
Changed lines of the file:
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@@
     (thickness 1.6)
     (drawings 1)
-    (tracks 398)
+    (tracks 449)
     (zones 0)
     (modules 319)
@@
   (via (at 181.35 12.329999) (size 0.6) (drill 0.3) (layers F.Cu B.Cu) (net 1))
   (via (at 188 13.829999) (size 0.6) (drill 0.3) (layers F.Cu B.Cu) (net 1))
+  (via (at 16.299999 4.7) (size 0.6) (drill 0.3) (layers F.Cu B.Cu) (net 1))
+  (via (at 27.049999 4.7) (size 0.6) (drill 0.3) (layers F.Cu B.Cu) (net 1))
+  (via (at 37.8 4.7) (size 0.6) (drill 0.3) (layers F.Cu B.Cu) (net 1))
+  (via (at 48.55 4.7) (size 0.6) (drill 0.3) (layers F.Cu B.Cu) (net 1))
+  (via (at 59.3 4.7) (size 0.6) (drill 0.3) (layers F.Cu B.Cu) (net 1))
+  (via (at 70.05 4.7) (size 0.6) (drill 0.3) (layers F.Cu B.Cu) (net 1))
   (via (at 67.125 75.49) (size 0.6) (drill 0.3) (layers F.Cu B.Cu) (net 1))
+  (via (at 48.099999 66.454999) (size 0.6) (drill 0.3) (layers F.Cu B.Cu) (net 1))
+  (via (at 14.349999 5.2) (size 0.6) (drill 0.3) (layers F.Cu B.Cu) (net 1))
   (via (at 2.9 4.45) (size 0.6) (drill 0.3) (layers F.Cu B.Cu) (net 1))
   (via (at 130.309999 73.374998) (size 0.6) (drill 0.3) (layers F.Cu B.Cu) (net 1))
@@
   (via (at 181.35 9.429998) (size 0.6) (drill 0.3) (layers F.Cu B.Cu) (net 1))
   (via (at 185.7 13.829999) (size 0.6) (drill 0.3) (layers F.Cu B.Cu) (net 1))
+  (via (at 18.599999 2.9) (size 0.6) (drill 0.3) (layers F.Cu B.Cu) (net 1))
+  (via (at 29.349999 2.9) (size 0.6) (drill 0.3) (layers F.Cu B.Cu) (net 1))
+  (via (at 40.099999 2.9) (size 0.6) (drill 0.3) (layers F.Cu B.Cu) (net 1))
+  (via (at 50.849999 2.9) (size 0.6) (drill 0.3) (layers F.Cu B.Cu) (net 1))
+  (via (at 61.599999 2.9) (size 0.6) (drill 0.3) (layers F.Cu B.Cu) (net 1))
+  (via (at 72.35 2.9) (size 0.6) (drill 0.3) (layers F.Cu B.Cu) (net 1))
   (via (at 67.125 73.39) (size 0.6) (drill 0.3) (layers F.Cu B.Cu) (net 1))
+  (via (at 48.099999 63.054998) (size 0.6) (drill 0.3) (layers F.Cu B.Cu) (net 1))
+  (via (at 10.3 9.249999) (size 0.6) (drill 0.3) (layers F.Cu B.Cu) (net 1))
+  (via (at 5.199999 2.9) (size 0.6) (drill 0.3) (layers F.Cu B.Cu) (net 1))
   (via (at 130.084256 75.555249) (size 0.6) (drill 0.3) (layers F.Cu B.Cu) (net 1))
   (via (at 134.744257 75.555249) (size 0.6) (drill 0.3) (layers F.Cu B.Cu) (net 1))
@@
   (via (at 149.05 65.604999) (size 0.6) (drill 0.3) (layers F.Cu B.Cu) (net 2))
   (via (at 144.95 65.604999) (size 0.6) (drill 0.3) (layers F.Cu B.Cu) (net 2))
+  (via (at 164.16 33.104999) (size 0.6) (drill 0.3) (layers F.Cu B.Cu) (net 2))
   (via (at 173.86 20.039999) (size 0.6) (drill 0.3) (layers F.Cu B.Cu) (net 2))
   (via (at 147.36 46.169999) (size 0.6) (drill 0.3) (layers F.Cu B.Cu) (net 2))
@@
   (via (at 183.15 10.879999) (size 0.6) (drill 0.3) (layers F.Cu B.Cu) (net 2))
   (via (at 188 10.879999) (size 0.6) (drill 0.3) (layers F.Cu B.Cu) (net 2))
+  (via (at 22.799999 4.7) (size 0.6) (drill 0.3) (layers F.Cu B.Cu) (net 2))
+  (via (at 33.549999 4.7) (size 0.6) (drill 0.3) (layers F.Cu B.Cu) (net 2))
+  (via (at 44.3 4.7) (size 0.6) (drill 0.3) (layers F.Cu B.Cu) (net 2))
+  (via (at 55.05 4.7) (size 0.6) (drill 0.3) (layers F.Cu B.Cu) (net 2))
+  (via (at 65.8 4.7) (size 0.6) (drill 0.3) (layers F.Cu B.Cu) (net 2))
+  (via (at 76.55 4.7) (size 0.6) (drill 0.3) (layers F.Cu B.Cu) (net 2))
   (via (at 70.475 75.49) (size 0.6) (drill 0.3) (layers F.Cu B.Cu) (net 2))
+  (via (at 52.399999 66.454999) (size 0.6) (drill 0.3) (layers F.Cu B.Cu) (net 2))
+  (via (at 100.45 53.469998) (size 0.6) (drill 0.3) (layers F.Cu B.Cu) (net 2))
   (via (at 119.669999 21.249999) (size 0.6) (drill 0.3) (layers F.Cu B.Cu) (net 2))
   (via (at 110.974999 18.014999) (size 0.6) (drill 0.3) (layers F.Cu B.Cu) (net 2))
@@
   (via (at 126 51.629999) (size 0.6) (drill 0.3) (layers F.Cu B.Cu) (net 2))
   (via (at 117.35 51.629999) (size 0.6) (drill 0.3) (layers F.Cu B.Cu) (net 2))
+  (via (at 127 49.999999) (size 0.6) (drill 0.3) (layers F.Cu B.Cu) (net 2))
+  (via (at 118.35 49.999999) (size 0.6) (drill 0.3) (layers F.Cu B.Cu) (net 2))
   (via (at 124.424328 49.648459) (size 0.6) (drill 0.3) (layers F.Cu B.Cu) (net 2))
   (via (at 124.424328 46.241538) (size 0.6) (drill 0.3) (layers F.Cu B.Cu) (net 2))
@@
   (via (at 147.05 65.604999) (size 0.6) (drill 0.3) (layers F.Cu B.Cu) (net 2))
   (via (at 143.95 66.654999) (size 0.6) (drill 0.3) (layers F.Cu B.Cu) (net 2))
+  (via (at 160.61 36.654999) (size 0.6) (drill 0.3) (layers F.Cu B.Cu) (net 2))
   (via (at 172.31 21.039999) (size 0.6) (drill 0.3) (layers F.Cu B.Cu) (net 2))
   (via (at 148.91 45.169999) (size 0.6) (drill 0.3) (layers F.Cu B.Cu) (net 2))
@@
   (via (at 99.525 69.44) (size 0.6) (drill 0.3) (layers F.Cu B.Cu) (net 2))
   (via (at 103.625 69.44) (size 0.6) (drill 0.3) (layers F.Cu B.Cu) (net 2))
+  (via (at 60.155483 66.076295) (size 0.6) (drill 0.3) (layers F.Cu B.Cu) (net 2))
+  (via (at 66.555483 66.076295) (size 0.6) (drill 0.3) (layers F.Cu B.Cu) (net 2))
+  (via (at 72.955483 66.076295) (size 0.6) (drill 0.3) (layers F.Cu B.Cu) (net 2))
+  (via (at 79.355484 66.076295) (size 0.6) (drill 0.3) (layers F.Cu B.Cu) (net 2))
+  (via (at 85.755484 66.076295) (size 0.6) (drill 0.3) (layers F.Cu B.Cu) (net 2))
+  (via (at 92.155484 66.076295) (size 0.6) (drill 0.3) (layers F.Cu B.Cu) (net 2))
+  (via (at 98.555484 66.076295) (size 0.6) (drill 0.3) (layers F.Cu B.Cu) (net 2))
   (via (at 114.96 73.374998) (size 0.6) (drill 0.3) (layers F.Cu B.Cu) (net 2))
   (via (at 47.025 73.39) (size 0.6) (drill 0.3) (layers F.Cu B.Cu) (net 2))
+  (via (at 104.955484 66.076295) (size 0.6) (drill 0.3) (layers F.Cu B.Cu) (net 2))
+  (via (at 111.355484 66.076295) (size 0.6) (drill 0.3) (layers F.Cu B.Cu) (net 2))
   (via (at 119.62 73.374998) (size 0.6) (drill 0.3) (layers F.Cu B.Cu) (net 2))
   (via (at 53.725 73.39) (size 0.6) (drill 0.3) (layers F.Cu B.Cu) (net 2))
+  (via (at 117.755484 66.076295) (size 0.6) (drill 0.3) (layers F.Cu B.Cu) (net 2))
+  (via (at 124.155484 66.076295) (size 0.6) (drill 0.3) (layers F.Cu B.Cu) (net 2))
   (via (at 124.604919 73.382291) (size 0.6) (drill 0.3) (layers F.Cu B.Cu) (net 2))
   (via (at 60.425 73.39) (size 0.6) (drill 0.3) (layers F.Cu B.Cu) (net 2))
+  (via (at 130.555484 66.076295) (size 0.6) (drill 0.3) (layers F.Cu B.Cu) (net 2))
+  (via (at 136.955484 66.076295) (size 0.6) (drill 0.3) (layers F.Cu B.Cu) (net 2))
   (via (at 173.3 12.329999) (size 0.6) (drill 0.3) (layers F.Cu B.Cu) (net 2))
   (via (at 178.8 12.329999) (size 0.6) (drill 0.3) (layers F.Cu B.Cu) (net 2))
   (via (at 184.3 12.329999) (size 0.6) (drill 0.3) (layers F.Cu B.Cu) (net 2))
   (via (at 186.85 9.429998) (size 0.6) (drill 0.3) (layers F.Cu B.Cu) (net 2))
+  (via (at 20.499999 2.9) (size 0.6) (drill 0.3) (layers F.Cu B.Cu) (net 2))
+  (via (at 31.249999 2.9) (size 0.6) (drill 0.3) (layers F.Cu B.Cu) (net 2))
+  (via (at 42 2.9) (size 0.6) (drill 0.3) (layers F.Cu B.Cu) (net 2))
+  (via (at 52.75 2.9) (size 0.6) (drill 0.3) (layers F.Cu B.Cu) (net 2))
+  (via (at 63.5 2.9) (size 0.6) (drill 0.3) (layers F.Cu B.Cu) (net 2))
+  (via (at 74.25 2.9) (size 0.6) (drill 0.3) (layers F.Cu B.Cu) (net 2))
   (via (at 70.475 73.39) (size 0.6) (drill 0.3) (layers F.Cu B.Cu) (net 2))
+  (via (at 52.399999 63.054998) (size 0.6) (drill 0.3) (layers F.Cu B.Cu) (net 2))
+  (via (at 100.45 46.369999) (size 0.6) (drill 0.3) (layers F.Cu B.Cu) (net 2))
   (via (at 119.669999 19.449999) (size 0.6) (drill 0.3) (layers F.Cu B.Cu) (net 2))
   (via (at 110.974999 15.914998) (size 0.6) (drill 0.3) (layers F.Cu B.Cu) (net 2))
@@
   (via (at 164.325 14.764999) (size 0.6) (drill 0.3) (layers F.Cu B.Cu) (net 2))
   (via (at 97.774999 58.62) (size 0.6) (drill 0.3) (layers F.Cu B.Cu) (net 2))
+  (via (at 181.659999 71.464999) (size 0.6) (drill 0.3) (layers F.Cu B.Cu) (net 2))
   (zone (net 0) (net_name "") (layers F.Cu In1.Cu In2.Cu In3.Cu In4.Cu B.Cu) (hatch edge 0.508)
     (connect_pads (clearance 0.3))
